File: _autosave-rnm-75E.kicad_pcb (KiCad board)
At the start: 2 copper layers, 93.7 x 38.1 mm, 24 parts, among them SW1 SW_Push, U1 ATmega32U4-AU, Y1 Crystal_GND24_Small

Commit message: ROUTED
Parts:
- moved D2 10.2 mm to (130.2, 125.5), turned to 90 degrees
- moved D4 10.0 mm to (149.1, 125.5), turned to 90 degrees
- moved D1 9.97 mm to (130.2, 106.7), turned to 90 degrees
- moved D3 9.87 mm to (149.1, 106.7), turned to 90 degrees
- moved R3 8.37 mm to (181.0, 115.8), turned to 90 degrees
- moved C7 4.70 mm to (180.5, 108.8), turned to 90 degrees
Connections:
- U1 pad 26: Net-(U1-Pad26) -> ROW1
- U1 pad 30: ROW1 -> Net-(U1-Pad30)
Routing:
- net +5V: track 88.7 -> 161.8 mm, vias 4 -> 3
- net COL1: track 0.00 -> 52.2 mm
- net ROW1: track 0.00 -> 51.6 mm
- net GND: track 100.8 -> 149.6 mm
- net ROW0: track 0.00 -> 38.8 mm
- net COL0: track 0.00 -> 19.0 mm
- net Net-(D1-Pad2): track 0.00 -> 8.09 mm
- net Net-(D3-Pad2): track 0.00 -> 8.04 mm
- net Net-(D2-Pad2): track 0.00 -> 7.91 mm
- net Net-(D4-Pad2): track 0.00 -> 7.71 mm
- net Net-(C7-Pad1): track 10.8 -> 7.24 mm
