File: rnm-75E.sch (KiCad schematic (older format))
At the start: 197 parts

Commit message: place encoder
Parts:
- added D?: D_Small, symbol Device:D_Small
- added SW?: Rotary_Encoder_Switch, symbol Device:Rotary_Encoder_Switch
Connections:
- net COL13: now also U?.8 (PB0); no longer U?.11 (PB3)
- net COL14: now also U?.1 (PE6); no longer U?.10 (PB2)
- net COL15: now also SW?.S1
- net MISO: now also U?.11 (PB3); no longer U?.8 (PB0)
- net MOSI: now also U?.10 (PB2); no longer U?.9 (PB1)
- net ROWA: now also D?.1 (K)
- net SCK: now also U?.9 (PB1); no longer U?.1 (PE6)
- new net: D?.2 (A), SW?.S2
Changed lines of the file:
@@
 Wire Wire Line
 	6150 3600 5950 3600
-Text GLabel 10050 3500 2    50   Input ~ 0
+Text GLabel 10050 1400 2    50   Input ~ 0
 SCK
-Text GLabel 10050 1400 2    50   Input ~ 0
+Text GLabel 10050 1500 2    50   Input ~ 0
 MOSI
 Wire Wire Line
 	10500 3400 10050 3400
-Text GLabel 10050 1300 2    50   Input ~ 0
+Text GLabel 10050 1600 2    50   Input ~ 0
 MISO
 Text Notes 4500 0    0    50   ~ 0
@@
 Connection ~ 22300 1600
 Wire Wire Line
-	22300 1600 22300 250
+	22300 1600 22300 500
 Connection ~ 22300 2600
 Wire Wire Line
@@
 Text GLabel 10050 2500 2    50   Input ~ 0
 COL12
-Text GLabel 10050 1600 2    50   Input ~ 0
+Text GLabel 10050 1300 2    50   Input ~ 0
 COL13
-Text GLabel 10050 1500 2    50   Input ~ 0
+Text GLabel 10050 3500 2    50   Input ~ 0
 COL14
 Text GLabel 10050 2000 2    50   Input ~ 0
 COL15
+$Comp
+L Device:Rotary_Encoder_Switch SW?
+U 1 1 61694078
+P 21700 600
+F 0 "SW?" H 21700 967 50  0000 C CNN
+F 1 "Rotary_Encoder_Switch" H 21700 876 50  0000 C CNN
+F 2 "" H 21550 760 50  0001 C CNN
+F 3 "~" H 21700 860 50  0001 C CNN
+	1    21700 600
+	1    0    0    -1
+$EndComp
+$Comp
+L Device:D_Small D?
+U 1 1 6169EE37
+P 22000 900
+F 0 "D?" V 22046 830 50  0000 R CNN
+F 1 "D_Small" V 21955 830 50  0000 R CNN
+F 2 "" V 22000 900 50  0001 C CNN
+F 3 "~" V 22000 900 50  0001 C CNN
+	1    22000 900
+	0    -1   -1   0
+$EndComp
+Wire Wire Line
+	22000 500  22300 500
+Connection ~ 22300 500
+Wire Wire Line
+	22300 500  22300 250
+Wire Wire Line
+	22000 700  22000 800
+Wire Wire Line
+	22000 1000 20500 1000
+Connection ~ 20500 1000
 $EndSCHEMATC

Commit message: update mcu
Parts:
- added U1: AT90USB646-AU, Package_QFP:TQFP-64_14x14mm_P0.8mm, symbol MCU_Microchip_AVR:AT90USB646-AU
- gave numbers to parts that had none: 184
- renumbered C_FM to C_FM1, C_ucap to C_ucap1
Connections:
- net +5V: now also U1.21 (VCC), U1.3 (UVCC), U1.52 (VCC), U1.64 (AVCC), U1.8 (VBUS); no longer U2.14 (VCC), U2.2 (UVCC), U2.24 (AVCC), U2.34 (VCC), U2.44 (AVCC), U2.7 (VBUS)
- net COL0: now also U1.44 (PA7); no longer U2.32 (PC7)
- net COL1: now also U1.45 (PA6); no longer U2.31 (PC6)
- net COL10: now also U1.56 (PF5); no longer U2.20 (PD2)
- net COL11: now also U1.57 (PF4); no longer U2.19 (PD1)
- net COL12: now also U1.58 (PF3); no longer U2.18 (PD0)
- net COL13: now also U1.59 (PF2); no longer U2.8 (PB0)
- net COL14: now also U1.60 (PF1); no longer U2.1 (PE6)
- net COL15: now also U1.61 (PF0); no longer U2.12 (PB7)
- net COL2: now also U1.46 (PA5); no longer U2.30 (PB6)
- net COL3: now also U1.47 (PA4); no longer U2.29 (PB5)
- net COL4: now also U1.48 (PA3); no longer U2.28 (PB4)
- net COL5: now also U1.49 (PA2); no longer U2.27 (PD7)
- net COL6: now also U1.50 (PA1); no longer U2.26 (PD6)
- net COL7: no longer U2.25 (PD4)
- net COL8: now also U1.54 (PF7); no longer U2.22 (PD5)
- net COL9: now also U1.55 (PF6); no longer U2.21 (PD3)
- net D+: now also U1.5 (D+); no longer U2.4 (D+)
- net D-: now also U1.4 (D-); no longer U2.3 (D-)
- net GND: now also R_SW2.2, U1.22 (GND), U1.53 (GND), U1.6 (UGND), U1.63 (GND); no longer R_SW2.1, U2.15 (GND), U2.23 (GND), U2.35 (GND), U2.43 (GND), U2.5 (UGND)
- net MISO: now also U1.13 (PB3); no longer U2.11 (PB3)
- net MOSI: now also U1.12 (PB2); no longer U2.10 (PB2)
- net RESET: now also U1.20 (~RESET); no longer U2.13 (~RESET)
- net ROWA: now also U1.30 (PD5); no longer U2.36 (PF7)
- net ROWB: now also U1.29 (PD4); no longer U2.37 (PF6)
- net ROWC: now also U1.28 (PD3); no longer U2.38 (PF5)
- net ROWD: now also U1.27 (PD2); no longer U2.39 (PF4)
- net ROWE: now also U1.26 (PD1); no longer U2.40 (PF1)
- net ROWF: now also U1.25 (PD0); no longer U2.41 (PF0)
- net SCK: now also U1.11 (PB1); no longer U2.9 (PB1)
- net XTAL1: now also U1.24 (XTAL1); no longer U2.17 (XTAL1)
- net XTAL2: now also U1.23 (XTAL2); no longer U2.16 (XTAL2)
- net at U2.33 (~HWB~/PE2): no longer R_SW2.2
- net at U2.6 (UCAP): no longer C_ucap1.2
- new net: U2.14 (VCC), U2.34 (VCC)
- new net: U2.15 (GND), U2.23 (GND), U2.35 (GND), U2.43 (GND)
- new net: U2.24 (AVCC), U2.44 (AVCC)
- new net: C_ucap1.2, U1.7 (UCAP)
- new net: R_SW2.1, U1.43 (PE2/~HWB)
Other:
- note removed: "MISO and MOSI are good on 8/9 or 10/11. 13 is RESET 12 is on another bank. 7 5v 8-11 good"
- moved on the sheet: CF3, C_F1, C_F2, C_F4, C_FM1, C_ucap1, R_SW2, U2
