File: _autosave-rnm-75E.sch (KiCad schematic (older format))
At the start: 212 parts, among them J1 AVR-ISP-6, J2 USB_C_Receptacle_USB2.0, J3 Conn_01x04, SW1 SW_Push, SW2 Rotary_Encoder_Switch, U1 AT90USB646-AU, Y1 Crystal_GND24_Small

Commit message: Added TODO
Parts:
- added MX90: MX-NoLED, MX_ONLY:MXOnly-1.25U-NoLED, symbol MX_ALPS_HYBRID:MX-NoLED
Connections:
- net COL1: now also MX90.1 (COL)
- net at D9.2 (A), MX9.2 (ROW): now also MX90.2 (ROW)
Other:
- note added: "ADD STEPPED CAPS SUPPORT\nUSES STEM PLACEMENT INLINE WITH L-CTRL\n"
Changed lines of the file:
@@
 Connection ~ 13150 8450
 Wire Wire Line
-	13150 8450 13150 7450
+	13150 8450 13150 8100
 Connection ~ 13150 9450
 Wire Wire Line
@@
 Text GLabel 4500 9700 2    50   Input ~ 0
 SDA
+Text Notes 9300 8250 0    50   ~ 0
+ADD STEPPED CAPS SUPPORT\nUSES STEM PLACEMENT INLINE WITH L-CTRL\n
+$Comp
+L MX_ALPS_HYBRID:MX-NoLED MX90
+U 1 1 60E8593B
+P 12650 8450
+F 0 "MX90" H 12650 8600 60  0000 C CNN
+F 1 "MX-NoLED" V 12500 8450 20  0000 C CNN
+F 2 "MX_ONLY:MXOnly-1.25U-NoLED" H 12025 8425 60  0001 C CNN
+F 3 "" H 12025 8425 60  0001 C CNN
+	1    12650 8450
+	1    0    0    -1
+$EndComp
+Wire Wire Line
+	13150 8100 12800 8100
+Wire Wire Line
+	12800 8100 12800 8400
+Connection ~ 13150 8100
+Wire Wire Line
+	13150 8100 13150 7450
+Wire Wire Line
+	12600 8600 12850 8600
+Wire Wire Line
+	12850 8600 12850 8650
+Connection ~ 12850 8650
 $EndSCHEMATC
