File: _autosave-rnm-75E.sch (KiCad schematic (older format))
At the start: 218 parts, among them J1 AVR-ISP-6, J2 USB_C_Receptacle_USB2.0, J3 Conn_01x04, SW1 SW_Push, SW2 Rotary_Encoder_Switch, U1 AT90USB1286-AU, U2 SRV05-4, Y1 Crystal_GND24_Small

Commit message: rerun main ground
Parts:
- added C_F3: 0.1uF, Capacitor_SMD:C_0805_2012Metric, symbol Device:C_Small
Connections:
- net +5V: now also C_F3.2
- net GND: now also C_F3.1
Changed lines of the file:
@@
 Wire Wire Line
 	4850 4650 4850 4200
+$Comp
+L Device:C_Small C_F3
+U 1 1 60A3A0B9
+P 5650 6200
+F 0 "C_F3" H 5742 6246 50  0000 L CNN
+F 1 "0.1uF" H 5742 6155 50  0000 L CNN
+F 2 "Capacitor_SMD:C_0805_2012Metric" H 5650 6200 50  0001 C CNN
+F 3 "~" H 5650 6200 50  0001 C CNN
+	1    5650 6200
+	1    0    0    1
+$EndComp
+Wire Wire Line
+	6050 6100 5650 6100
+Connection ~ 6050 6100
+Wire Wire Line
+	5650 6300 6050 6300
+Connection ~ 6050 6300
 $EndSCHEMATC

Commit message: autosave hro
Parts:
- J2: footprint Connector_USB:USB_C_Receptacle_Palconn_UTC16-G -> Connector_USB:USB_C_Receptacle_HRO_TYPE-C-31-M-12
Changed lines of the file:
@@
 F 0 "J2" H 2057 5867 50  0000 C CNN
 F 1 "USB_C_Receptacle_USB2.0" H 2057 5776 50  0000 C CNN
-F 2 "Connector_USB:USB_C_Receptacle_Palconn_UTC16-G" H 2100 5000 50  0001 C CNN
+F 2 "Connector_USB:USB_C_Receptacle_HRO_TYPE-C-31-M-12" H 2100 5000 50  0001 C CNN
 F 3 "https://www.usb.org/sites/default/files/documents/usb_type-c.zip" H 2100 5000 50  0001 C CNN
 	1    1950 5000
