File: rnm-75E.kicad_pcb (KiCad board)
At the start: 2 copper layers, 323.8 x 114.3 mm, 217 parts, among them J1 AVR-ISP-6, J2 USB_C_Receptacle_USB2.0, J3 Conn_01x04, SW1 SW_Push, SW2 Rotary_Encoder_Switch, U1 AT90USB646-AU, Y1 Crystal_GND24_Small

Commit message: visual changes
Parts:
- moved D93 1.48 mm to (629.8, -7.29)
Changed lines of the file:
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@@
     (thickness 1.6)
     (drawings 8)
-    (tracks 1458)
+    (tracks 1460)
     (zones 0)
     (modules 217)
@@
   )
   (module LED_SMD:LED_WS2812B_PLCC4_5.0x5.0mm_P3.2mm (layer B.Cu)
-    (at 630.9625 -6.3375)
+    (at 629.83 -7.29)
     (descr https://cdn-shop.adafruit.com/datasheets/WS2812B.pdf)
     (tags "LED RGB NeoPixel")
@@
   (segment (start 618.39375 6.35) (end 619.91875 4.825) (width 0.254) (layer B.Cu) (net 21))
   (segment (start 593.09 6.35) (end 618.39375 6.35) (width 0.254) (layer B.Cu) (net 21))
-  (via (at 621.03 6.35) (size 0.8) (drill 0.4) (layers F.Cu B.Cu) (net 21))
   (segment (start 619.91875 5.23875) (end 621.03 6.35) (width 0.254) (layer B.Cu) (net 21))
   (segment (start 619.91875 4.825) (end 619.91875 5.23875) (width 0.254) (layer B.Cu) (net 21))
-  (segment (start 621.03 6.35) (end 631.19 6.35) (width 0.254) (layer F.Cu) (net 21))
-  (via (at 631.19 6.35) (size 0.8) (drill 0.4) (layers F.Cu B.Cu) (net 21))
   (segment (start 648.49375 4.825) (end 648.49375 5.55625) (width 0.254) (layer B.Cu) (net 21))
   (segment (start 647.7 6.35) (end 631.19 6.35) (width 0.254) (layer B.Cu) (net 21))
@@
   (segment (start 495.506253 70.850003) (end 488.95 70.850003) (width 0.254) (layer B.Cu) (net 21))
   (segment (start 498.0625 73.40625) (end 495.506253 70.850003) (width 0.254) (layer B.Cu) (net 21))
+  (via (at 624.84 6.35) (size 0.8) (drill 0.4) (layers F.Cu B.Cu) (net 21))
+  (segment (start 621.03 6.35) (end 624.84 6.35) (width 0.254) (layer B.Cu) (net 21))
+  (via (at 629.92 6.35) (size 0.8) (drill 0.4) (layers F.Cu B.Cu) (net 21))
+  (segment (start 631.19 6.35) (end 629.92 6.35) (width 0.254) (layer B.Cu) (net 21))
+  (segment (start 629.92 6.35) (end 624.84 6.35) (width 0.254) (layer F.Cu) (net 21))
   (segment (start 608.80625 23.875) (end 608.585 23.875) (width 0.254) (layer B.Cu) (net 22))
   (segment (start 608.585 23.875) (end 607.06 25.4) (width 0.254) (layer B.Cu) (net 22))

Commit message: neater route 13
Routing:
- net COL13: track 218.5 -> 195.6 mm
Changed lines of the file:
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@@
   (segment (start 515.7 79.00625) (end 517.15625 79.00625) (width 0.254) (layer B.Cu) (net 136))
   (segment (start 589.12125 49.37125) (end 589.12125 19.685) (width 0.254) (layer F.Cu) (net 136))
-  (segment (start 611.98125 61.9125) (end 602.45625 52.3875) (width 0.254) (layer F.Cu) (net 136))
-  (segment (start 602.45625 52.3875) (end 592.1375 52.3875) (width 0.254) (layer F.Cu) (net 136))
-  (segment (start 611.98125 79.375) (end 611.98125 61.9125) (width 0.254) (layer F.Cu) (net 136))
-  (segment (start 591.982326 82.55) (end 608.80625 82.55) (width 0.254) (layer F.Cu) (net 136))
+  (segment (start 592.954501 53.204501) (end 589.12125 49.37125) (width 0.254) (layer F.Cu) (net 136))
+  (segment (start 600.098251 74.318251) (end 592.954501 67.174501) (width 0.254) (layer F.Cu) (net 136))
+  (segment (start 591.982326 82.55) (end 596.9 82.55) (width 0.254) (layer F.Cu) (net 136))
   (segment (start 591.474396 83.05793) (end 591.982326 82.55) (width 0.254) (layer F.Cu) (net 136))
   (segment (start 535.026204 83.05793) (end 591.474396 83.05793) (width 0.254) (layer F.Cu) (net 136))
-  (segment (start 608.80625 82.55) (end 611.98125 79.375) (width 0.254) (layer F.Cu) (net 136))
+  (segment (start 592.954501 67.174501) (end 592.954501 53.204501) (width 0.254) (layer F.Cu) (net 136))
   (segment (start 532.753803 80.785529) (end 535.026204 83.05793) (width 0.254) (layer F.Cu) (net 136))
-  (segment (start 592.1375 52.3875) (end 589.12125 49.37125) (width 0.254) (layer F.Cu) (net 136))
   (segment (start 529.57926 80.785529) (end 532.753803 80.785529) (width 0.254) (layer F.Cu) (net 136))
+  (segment (start 596.9 82.55) (end 600.098251 79.351749) (width 0.254) (layer F.Cu) (net 136))
+  (segment (start 600.098251 79.351749) (end 600.098251 74.318251) (width 0.254) (layer F.Cu) (net 136))
   (segment (start 616.10526 76.835) (end 617.69625 76.835) (width 0.254) (layer F.Cu) (net 137))
   (segment (start 614.045 76.835) (end 616.10526 76.835) (width 0.254) (layer F.Cu) (net 137))

Commit message: oled and top gnd
Parts:
- moved J3 1.12 mm to (616.7, -19.8)
Connections:
- F1 pad 2: ENCODER+ -> VCC
- J1 pad 2: ENCODER+ -> VCC
- J2 pad A4: ENCODER+ -> VCC
- J2 pad A9: ENCODER+ -> VCC
- J2 pad B4: ENCODER+ -> VCC
- J2 pad B9: ENCODER+ -> VCC
- SW2 pad B: ENCODER+ -> ENCODER-
- U1 pad 55: ENCODER+ -> ENCODER-
Routing:
- net GND: track 255.6 -> 630.7 mm
- net ENCODER+: track 560.1 -> 280.7 mm, vias 2 -> 1
- net ENCODER-: track 0.00 -> 274.9 mm, vias 0 -> 1
- net VCC: track 0.00 -> 21.2 mm, vias 0 -> 2
- net MOSI: track 204.9 -> 187.8 mm
- net +5V: track 350.3 -> 366.8 mm
- net SDA: track 244.7 -> 251.9 mm

Commit message: emcoder routing
Connections:
- U1 pad 54: ENCODER+ -> ENCODER-
- U1 pad 55: ENCODER- -> ENCODER+
Routing:
- net COL0: track 314.0 -> 324.8 mm
- net GND: track 630.7 -> 635.2 mm
- net ENCODER-: track 274.9 -> 278.5 mm
- net ENCODER+: track 280.7 -> 284.0 mm

Commit message: pretty
Parts:
- moved R_SW2 25.3 mm to (532.6, 85.8), turned to 90 degrees
- moved D97 2.21 mm to (419.2, 67.6), turned to 180 degrees
- moved J1 1.12 mm to (647.7, -3.97), turned to 270 degrees
- moved D89 0.07 mm to (345.4, -6.34)
- turned D93 to 180 degrees
- turned D94 to 270 degrees
- turned D95 to 180 degrees
- turned D96 to 180 degrees
- turned D98 to 180 degrees
Connections:
- D89 pad 4: LED -> Net-(D89-Pad4)
- D90 pad 2: Net-(D90-Pad2) -> Net-(D89-Pad4)
- D90 pad 4: Net-(D89-Pad2) -> Net-(D90-Pad4)
- D91 pad 2: Net-(D91-Pad2) -> Net-(D90-Pad4)
- D91 pad 4: Net-(D90-Pad2) -> Net-(D91-Pad4)
- D92 pad 2: Net-(D92-Pad2) -> Net-(D91-Pad4)
- D92 pad 4: Net-(D91-Pad2) -> Net-(D92-Pad4)
- D93 pad 2: Net-(D93-Pad2) -> Net-(D92-Pad4)
- D93 pad 4: Net-(D92-Pad2) -> Net-(D93-Pad4)
- D94 pad 2: Net-(D94-Pad2) -> Net-(D93-Pad4)
- D94 pad 4: Net-(D93-Pad2) -> Net-(D94-Pad4)
- D95 pad 2: Net-(D95-Pad2) -> Net-(D94-Pad4)
- D95 pad 4: Net-(D94-Pad2) -> LED
- D96 pad 2: Net-(D96-Pad2) -> (no net)
- D96 pad 4: Net-(D95-Pad2) -> Net-(D96-Pad4)
- D97 pad 2: Net-(D97-Pad2) -> Net-(D96-Pad4)
- D97 pad 4: Net-(D96-Pad2) -> Net-(D97-Pad4)
- D98 pad 2: (no net) -> Net-(D97-Pad4)
- D98 pad 4: Net-(D97-Pad2) -> Net-(D89-Pad2)
- SW2 pad C: GND -> (no net)
- U1 pad 10: LED -> (no net)
- U1 pad 42: (no net) -> LED
Routing:
- net +5V: track 366.8 -> 926.3 mm, vias 5 -> 10
- net RESET: track 70.9 -> 246.7 mm
- net Net-(D89-Pad2): track 0.00 -> 99.9 mm
- net Net-(D93-Pad4): track 0.00 -> 91.8 mm, vias 0 -> 2
- net LED: track 0.00 -> 78.0 mm
- net Net-(D91-Pad4): track 0.00 -> 76.1 mm
- net Net-(D90-Pad4): track 0.00 -> 74.2 mm
- net Net-(D89-Pad4): track 0.00 -> 71.8 mm
- net Net-(D97-Pad4): track 0.00 -> 71.2 mm
- net Net-(D92-Pad4): track 0.00 -> 62.7 mm
- net Net-(D94-Pad4): track 0.00 -> 55.3 mm
- net Net-(D96-Pad4): track 0.00 -> 54.2 mm
- net Net-(R_SW2-Pad1): track 0.00 -> 32.6 mm
- net MOSI: track 187.8 -> 176.3 mm
- net VCC: track 21.2 -> 15.3 mm, vias 2 -> 1
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
Commit message: add ISP
Routing:
- net MOSI: track 176.3 -> 190.1 mm, vias 0 -> 2
- net GND: track 635.5 -> 641.9 mm
- net VCC: track 15.3 -> 20.7 mm, vias 1 -> 2
- net SCK: track 188.3 -> 189.6 mm

Commit message: all mcu connected
Parts:
- turned C_F1 to 0 degrees
- turned C_F4 to 270 degrees
- turned C_FM1 to 0 degrees
Routing:
- net GND: track 641.9 -> 804.3 mm, vias 0 -> 4
- net +5V: track 926.3 -> 921.8 mm
- net D+: track 196.0 -> 196.7 mm
- net D-: track 195.7 -> 196.4 mm
- net ROWF: track 373.4 -> 372.8 mm

Commit message: added ground fill
Connections:
- U1 pad 10: (no net) -> LED_PIN
- U1 pad 9: LED_PIN -> (no net)
Routing:
- net GND: track 804.3 -> 1140.7 mm, vias 4 -> 6
- net +5V: track 921.8 -> 1011.3 mm, vias 10 -> 12
- net LED_PIN: track 263.2 -> 262.6 mm
- added copper zone on B.Cu, net GND
