File: PLATE/plate/plate.kicad_pcb (KiCad board)
At the start: 2 copper layers, 323.8 x 114.3 mm, 0 parts

Commit message: plate
Other:
- outline, holes or cut-outs redrawn
- board text added: "-Anthony Luo"

Commit message: gerber3
Other:
- outline, holes or cut-outs redrawn
- board text removed: "-Anthony Luo"

Commit message: plate3 gerbers
Routing:
- net (no net): track 0.00 -> 214.6 mm, vias 0 -> 2
Changed lines of the file:
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@@
     (thickness 1.6)
     (drawings 750)
-    (tracks 0)
+    (tracks 6)
     (zones 0)
     (modules 0)
@@
       (drillshape 0)
       (scaleselection 1)
-      (outputdirectory "D:/Keyboard_Designs/rnm-75E/PLATE/gerbers/"))
+      (outputdirectory "D:/Keyboard_Designs/rnm-75E/PLATE/gerbers3/"))
   )
   (net 0 "")
@@
   (gr_line (start 81.699 64.643) (end 81.699 77.643) (layer Edge.Cuts) (width 0.2))
   (gr_arc (start 68.199 64.643) (end 68.199 64.143) (angle -90) (layer Edge.Cuts) (width 0.2))
+  (segment (start 26.67 62.23) (end 26.67 62.23) (width 0.25) (layer B.Cu) (net 0))
+  (segment (start 170.095854 62.23) (end 241.3 62.23) (width 0.25) (layer B.Cu) (net 0))
+  (segment (start 241.3 62.23) (end 241.3 62.23) (width 0.25) (layer B.Cu) (net 0))
+  (via (at 241.3 62.23) (size 0.8) (drill 0.4) (layers F.Cu B.Cu) (net 0))
+  (segment (start 26.67 62.23) (end 170.095854 62.23) (width 0.25) (layer B.Cu) (net 0))
+  (via (at 26.67 62.23) (size 0.8) (drill 0.4) (layers F.Cu B.Cu) (net 0))
 )
